Commit message: feat: stage 3.3 diff drive, keyboard teleop, and VM-first git workflow
Add cmd_vel timeout relay with RELIABLE QoS, arrow-key teleop launch,
smoke test script, and git-based sync replacing destructive share-folder rsync.

Co-authored-by: Cursor <cursoragent@cursor.com>

File: ros2_ws/src/robot_description/urdf/robot_v0.gazebo.xacro (robot description, xacro)
@@ -1,6 +1,7 @@
 <?xml version="1.0"?>
 <!--
-  robot_v0 Gazebo 扩展（阶段 3.2）
-  仅物理/材质/摩擦参数，不含差速驱动插件（阶段 3.3 再加）
+  robot_v0 Gazebo 扩展
+  3.2：材质 / 摩擦 / 接触
+  3.3：差速驱动插件 + 关节状态发布（替代 joint_state_publisher 节点）
 -->
 <robot xmlns:xacro="http://www.ros.org/wiki/xacro">
@@ -29,7 +30,53 @@
   </gazebo>
   <gazebo reference="caster_link">
-    <material>Gazebo/Grey</material>
-    <mu1>0.05</mu1>
-    <mu2>0.05</mu2>
+    <material>Gazebo/Orange</material>
+    <mu1>0.1</mu1>
+    <mu2>0.1</mu2>
+    <kp>1000000.0</kp>
+    <kd>100.0</kd>
+  </gazebo>
+  <!-- 轮关节阻尼：静止时减少落地后「自己往前溜」 -->
+  <gazebo reference="left_wheel_joint">
+    <physics>
+      <ode>
+        <implicit_spring_damper>true</implicit_spring_damper>
+      </ode>
+    </physics>
+  </gazebo>
+  <gazebo reference="right_wheel_joint">
+    <physics>
+      <ode>
+        <implicit_spring_damper>true</implicit_spring_damper>
+      </ode>
+    </physics>
+  </gazebo>
+  <!-- 从仿真读取真实轮转角 → /joint_states -->
+  <gazebo>
+    <plugin name="gazebo_ros_joint_state_publisher"
+            filename="libgazebo_ros_joint_state_publisher.so">
+      <update_rate>50</update_rate>
+      <joint_name>left_wheel_joint</joint_name>
+      <joint_name>right_wheel_joint</joint_name>
+    </plugin>
+  </gazebo>
+  <!-- 差速驱动：/cmd_vel_gazebo → 轮子；/odom + odom→base_footprint TF -->
+  <gazebo>
+    <plugin name="diff_drive" filename="libgazebo_ros_diff_drive.so">
+      <ros>
+        <remapping>cmd_vel:=cmd_vel_gazebo</remapping>
+      </ros>
+      <left_joint>left_wheel_joint</left_joint>
+      <right_joint>right_wheel_joint</right_joint>
+      <wheel_separation>${wheel_separation}</wheel_separation>
+      <wheel_diameter>${2 * wheel_radius}</wheel_diameter>
+      <max_wheel_torque>20</max_wheel_torque>
+      <max_wheel_acceleration>1.0</max_wheel_acceleration>
+      <odometry_topic>odom</odometry_topic>
+      <odometry_frame>odom</odometry_frame>
+      <robot_base_frame>base_footprint</robot_base_frame>
+      <publish_odom>true</publish_odom>
+      <publish_odom_tf>true</publish_odom_tf>
+      <publish_wheel_tf>false</publish_wheel_tf>
+    </plugin>
   </gazebo>
 </robot>

File: ros2_ws/src/robot_description/urdf/robot_v0.urdf.xacro (robot description, xacro)
@@ -20,7 +20,10 @@
   <xacro:property name="wheel_mass" value="0.5"/>
   <xacro:property name="wheel_separation" value="0.28"/>
-  <xacro:property name="caster_radius" value="0.025"/>
-  <xacro:property name="caster_mass" value="0.1"/>
-  <xacro:property name="caster_offset_x" value="-0.12"/>
+  <!-- 驱动轮在车尾（-X）：与车头万向轮形成「后驱三轮」稳定布局 -->
+  <xacro:property name="wheel_offset_x" value="-0.12"/>
+  <xacro:property name="caster_radius" value="0.03"/>
+  <xacro:property name="caster_mass" value="0.2"/>
+  <!-- 万向轮在车头（+X） -->
+  <xacro:property name="caster_offset_x" value="0.14"/>
   <!-- base_link 中心离地高度 = 轮半径 + 底盘半高 -->
   <xacro:property name="base_z" value="${wheel_radius + base_height / 2.0}"/>
@@ -134,6 +137,7 @@
     <parent link="base_link"/>
     <child link="left_wheel_link"/>
-    <origin xyz="0 ${wheel_separation / 2.0} ${wheel_center_z}" rpy="0 0 0"/>
+    <origin xyz="${wheel_offset_x} ${wheel_separation / 2.0} ${wheel_center_z}" rpy="0 0 0"/>
     <axis xyz="0 1 0"/>
+    <dynamics damping="1.0" friction="1.0"/>
   </joint>
   <!-- ========== 右驱动轮 ========== -->
@@ -160,8 +164,9 @@
     <parent link="base_link"/>
     <child link="right_wheel_link"/>
-    <origin xyz="0 ${-wheel_separation / 2.0} ${wheel_center_z}" rpy="0 0 0"/>
+    <origin xyz="${wheel_offset_x} ${-wheel_separation / 2.0} ${wheel_center_z}" rpy="0 0 0"/>
     <axis xyz="0 1 0"/>
+    <dynamics damping="1.0" friction="1.0"/>
   </joint>
-  <!-- ========== 后万向轮（阶段 3.1 固定关节，仅支撑不驱动） ========== -->
+  <!-- 万向轮在车头（+X）；与中部驱动轮形成三点支撑（Gazebo 3.2 落地关键） -->
   <link name="caster_link">
     <visual>

Commit message: feat: stage 3.4 lidar /scan and fix combo keyboard teleop
Add laser_link ray sensor, lidar_test world, RViz config, and smoke test.
Fix keyboard teleop so angular key repeat keeps linear axes alive under Linux TTY.

Co-authored-by: Cursor <cursoragent@cursor.com>

File: ros2_ws/src/robot_description/urdf/robot_v0.gazebo.xacro (robot description, xacro)
@@ -4,4 +4,5 @@
   3.2：材质 / 摩擦 / 接触
   3.3：差速驱动插件 + 关节状态发布（替代 joint_state_publisher 节点）
+  3.4：ray 激光 → /scan（sensor_msgs/LaserScan）
 -->
 <robot xmlns:xacro="http://www.ros.org/wiki/xacro">
@@ -35,4 +36,57 @@
     <kp>1000000.0</kp>
     <kd>100.0</kd>
+  </gazebo>
+  <gazebo reference="laser_link">
+    <material>Gazebo/Red</material>
+    <!--
+      ========== 阶段 3.4：2D 激光雷达 ==========
+      数据流：Gazebo ray 传感器 → libgazebo_ros_ray_sensor.so → /scan (LaserScan)
+      自车红点（常见问题）：
+        1) 传感器装在 link 几何中心，水平射线会先撞到雷达外壳 collision
+        2) range.min 太小，近距车身角点没被滤掉
+      修法：laser_link 不要 collision；传感器 pose 抬到圆柱顶面；min_range ≥ 车身半径
+      圆柱方向线条稀疏（正常现象）：
+        远处小障碍物占的角度小。例：r=0.15m、距离≈1.6m → 张角约 11° → 360 线里只有 ~11 根打到柱子上，
+        其余射线穿过空隙打到墙或打到 max_range，所以 Gazebo 里看起来「稀」。
+    -->
+    <sensor name="laser" type="ray">
+      <always_on>true</always_on>
+      <!-- Gazebo 里蓝色射线；调试可看，验收以 RViz /scan 为准 -->
+      <visualize>true</visualize>
+      <update_rate>10</update_rate>
+      <!-- 光心：圆柱顶面 + 额外抬高，扫描平面远离蓝色车身 -->
+      <pose>0 0 ${laser_height / 2.0 + laser_scan_z_offset} 0 0 0</pose>
+      <ray>
+        <scan>
+          <horizontal>
+            <!-- 360 条射线，水平 360°，约 1° 一条 -->
+            <samples>360</samples>
+            <resolution>1.0</resolution>
+            <min_angle>-3.14159</min_angle>
+            <max_angle>3.14159</max_angle>
+          </horizontal>
+        </scan>
+        <range>
+          <!-- 小于 min 的命中在 /scan 里会变成 inf，RViz 不画 -->
+          <min>${laser_scan_min_range}</min>
+          <max>12.0</max>
+          <resolution>0.01</resolution>
+        </range>
+        <noise>
+          <type>gaussian</type>
+          <mean>0.0</mean>
+          <stddev>0.01</stddev>
+        </noise>
+      </ray>
+      <plugin name="gazebo_ros_laser" filename="libgazebo_ros_ray_sensor.so">
+        <ros>
+          <!-- ~/out 是插件默认话题名，remap 成导航栈习惯的 /scan -->
+          <remapping>~/out:=scan</remapping>
+        </ros>
+        <output_type>sensor_msgs/LaserScan</output_type>
+        <!-- TF / 消息 header.frame_id -->
+        <frame_name>laser_link</frame_name>
+      </plugin>
+    </sensor>
   </gazebo>
   <!-- 轮关节阻尼：静止时减少落地后「自己往前溜」 -->

File: ros2_ws/src/robot_description/urdf/robot_v0.urdf.xacro (robot description, xacro)
@@ -7,5 +7,6 @@
             ├── left_wheel_link
             ├── right_wheel_link
-            └── caster_link（万向支撑轮）
+            ├── caster_link（万向支撑轮）
+            └── laser_link（阶段 3.4 激光雷达）
   单位：米（SI）
 -->
@@ -26,4 +27,20 @@
   <!-- 万向轮在车头（+X） -->
   <xacro:property name="caster_offset_x" value="0.14"/>
+  <!-- 激光：小圆柱装在车身上方偏前，光心 = laser_link -->
+  <xacro:property name="laser_radius" value="0.03"/>
+  <xacro:property name="laser_height" value="0.04"/>
+  <xacro:property name="laser_mass" value="0.1"/>
+  <!-- 相对 base_link 前移 5cm，让雷达略靠车头 -->
+  <xacro:property name="laser_offset_x" value="0.05"/>
+  <!-- 雷达中心 z = 底盘半高 + 雷达半高，使雷达底面刚好贴在车顶 -->
+  <xacro:property name="laser_offset_z" value="${base_height / 2.0 + laser_height / 2.0}"/>
+  <!--
+    /scan 的 range_min（Gazebo 插件用）。
+    小于此距离的命中 → /scan 里变 inf，RViz 不画。
+    取 0.30：大于雷达到车身外轮廓水平距离（约 0.25m），留余量避免车顶一圈红点。
+  -->
+  <xacro:property name="laser_scan_min_range" value="0.30"/>
+  <!-- 光心再抬高 3cm（在圆柱顶面之上），进一步远离车身碰撞体 -->
+  <xacro:property name="laser_scan_z_offset" value="0.03"/>
   <!-- base_link 中心离地高度 = 轮半径 + 底盘半高 -->
   <xacro:property name="base_z" value="${wheel_radius + base_height / 2.0}"/>
@@ -193,4 +210,27 @@
     <origin xyz="${caster_offset_x} 0 ${-(base_z - caster_radius)}" rpy="0 0 0"/>
   </joint>
+  <!-- ========== 激光雷达（阶段 3.4）：固定在车顶，frame_id = laser_link ========== -->
+  <!--
+    只保留 visual，不要 collision：
+    Gazebo ray 从 link 原点水平出射，若外壳带碰撞体，射线会先打到自己（你看到的车身红点）。
+    真机雷达同理：支架不参与测距，只有光心坐标有意义。
+  -->
+  <link name="laser_link">
+    <visual>
+      <origin xyz="0 0 0" rpy="0 0 0"/>
+      <geometry>
+        <cylinder radius="${laser_radius}" length="${laser_height}"/>
+      </geometry>
+      <material name="red">
+        <color rgba="0.9 0.1 0.1 1.0"/>
+      </material>
+    </visual>
+    <xacro:sphere_inertial mass="${laser_mass}" radius="${laser_radius}"/>
+  </link>
+  <joint name="laser_joint" type="fixed">
+    <parent link="base_link"/>
+    <child link="laser_link"/>
+    <origin xyz="${laser_offset_x} 0 ${laser_offset_z}" rpy="0 0 0"/>
+  </joint>
   <!-- Gazebo 物理参数（阶段 3.2+） -->
   <xacro:include filename="robot_v0.gazebo.xacro"/>

Commit message: fix: stage 3.5 bumper camera with identity sensor pose, close stage 3
Remove camera mount links and use a low front bumper camera_link on
base_link. Gazebo Classic camera optical axis is +X, so identity pose
fixes downward frustum; pitch=1.5708 was wrong. Update docs with GUI
acceptance, troubleshooting archive, and stage 4 handoff.

Co-authored-by: Cursor <cursoragent@cursor.com>

File: ros2_ws/src/robot_description/urdf/robot_v0.gazebo.xacro (robot description, xacro)
@@ -91,15 +91,12 @@
     </sensor>
   </gazebo>
-  <gazebo reference="camera_mount_link">
-    <material>Gazebo/Grey</material>
-  </gazebo>
   <gazebo reference="camera_link">
     <material>Gazebo/Black</material>
     <!--
-      Gazebo 光轴默认 -Z；pitch +90° → 朝 base +X。
-      pose 必须写在 <camera> 之前；joint 禁止写 rpy（合并后 visual/sensor 会分裂）。
+      Gazebo Classic 相机光轴沿传感器 +X；camera_link 与 base_link 同向，恒等 pose 即朝车头。
+      pose 写在 <camera> 之前；joint 禁止写 rpy。
     -->
     <sensor name="camera" type="camera">
-      <pose>0 0 0 0 1.57079632679 0</pose>
+      <pose>0 0 0 0 0 0</pose>
       <always_on>true</always_on>
       <update_rate>10</update_rate>

File: ros2_ws/src/robot_description/urdf/robot_v0.urdf.xacro (robot description, xacro)
@@ -9,7 +9,6 @@
             ├── caster_link（万向支撑轮）
             ├── laser_link（阶段 3.4 激光雷达）
-            └── camera_mount_link（阶段 3.5 相机支架，仅 visual）
-                  └── camera_link
-                        └── camera_optical_frame
+            └── camera_link（阶段 3.5 前保险杠低位相机）
+                  └── camera_optical_frame
   单位：米（SI）
 -->
@@ -50,12 +49,7 @@
   <xacro:property name="camera_depth" value="0.03"/>
   <xacro:property name="camera_mass" value="0.05"/>
-  <!-- 支架锚点（车顶靠后）+ 相机相对支架偏移 → 光心仍在 x=0.22 z=0.13 -->
-  <xacro:property name="camera_mount_x" value="0.17"/>
-  <xacro:property name="camera_mount_z" value="0.09"/>
-  <xacro:property name="camera_rel_x" value="0.05"/>
-  <xacro:property name="camera_rel_z" value="0.04"/>
-  <!-- 支架细杆尺寸（仅 visual，无 collision） -->
-  <xacro:property name="mount_pillar_h" value="0.04"/>
-  <xacro:property name="mount_arm_len" value="0.05"/>
+  <!-- 前保险杠低位相机：车头前立面 x=0.20 凸出半深；光心离地约 0.12m -->
+  <xacro:property name="camera_offset_x" value="0.215"/>
+  <xacro:property name="camera_offset_z" value="0.02"/>
   <!-- base_link 中心离地高度 = 轮半径 + 底盘半高 -->
   <xacro:property name="base_z" value="${wheel_radius + base_height / 2.0}"/>
@@ -248,36 +242,8 @@
     <origin xyz="${laser_offset_x} 0 ${laser_offset_z}" rpy="0 0 0"/>
   </joint>
-  <!-- ========== 相机支架 + 相机（阶段 3.5）========== -->
-  <!-- 支架仅 visual：不挡 LiDAR /scan，也不进相机 collision -->
-  <link name="camera_mount_link">
-    <!-- 立柱：锚点 z=0.09 向下接到车顶 z=0.05 -->
-    <visual name="mount_pillar">
-      <origin xyz="0 0 ${-mount_pillar_h / 2.0}" rpy="0 0 0"/>
-      <geometry>
-        <box size="0.012 0.012 ${mount_pillar_h}"/>
-      </geometry>
-      <material name="mount_gray">
-        <color rgba="0.35 0.35 0.38 1.0"/>
-      </material>
-    </visual>
-    <!-- 前探横臂：从立柱顶 toward camera（略上仰，在相机后方不进 FOV） -->
-    <visual name="mount_arm">
-      <origin xyz="${mount_arm_len / 2.0} 0 ${camera_rel_z / 2.0}" rpy="0 0 0"/>
-      <geometry>
-        <box size="${mount_arm_len} 0.010 0.010"/>
-      </geometry>
-      <material name="mount_gray_arm">
-        <color rgba="0.35 0.35 0.38 1.0"/>
-      </material>
-    </visual>
-  </link>
-  <joint name="camera_mount_joint" type="fixed">
-    <parent link="base_link"/>
-    <child link="camera_mount_link"/>
-    <origin xyz="${camera_mount_x} 0 ${camera_mount_z}" rpy="0 0 0"/>
-  </joint>
+  <!-- ========== 相机（阶段 3.5）：前保险杠低位，无 collision ========== -->
   <link name="camera_link">
     <visual>
-      <origin xyz="${camera_depth / 2.0} 0 0" rpy="0 0 0"/>
+      <origin xyz="0 0 0" rpy="0 0 0"/>
       <geometry>
         <box size="${camera_depth} ${camera_width} ${camera_height}"/>
@@ -290,7 +256,7 @@
   </link>
   <joint name="camera_joint" type="fixed">
-    <parent link="camera_mount_link"/>
+    <parent link="base_link"/>
     <child link="camera_link"/>
-    <origin xyz="${camera_rel_x} 0 ${camera_rel_z}" rpy="0 0 0"/>
+    <origin xyz="${camera_offset_x} 0 ${camera_offset_z}" rpy="0 0 0"/>
   </joint>
   <!-- ROS 光学系：Z 前、X 右、Y 下（阶段 5 YOLO/投影用；3.5 图像 frame_id 仍用 camera_link） -->
